Commit message: feat: cellule RViz complète - silo, contrôleur, ventilation, tête extrusion

File: ros2_ws/src/staubli_description/urdf/rx160l.urdf (robot description, URDF)
Before this commit: robot staubli_rx160l, 9 links, 8 joints
Links:
- added link aeration; visual mesh filename=package://staubli_description/meshes/visual/cell/aeration.s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 scale=0.001 0.001 0.001
- added link controleur; visual mesh filename=package://staubli_description/meshes/visual/cell/controleur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 scale=0.001 0.001 0.001
- added link silo; visual mesh filename=package://staubli_description/meshes/visual/cell/silo.stl scale=0.001 0.001 0.001
- added link tete_extrusion; visual mesh filename=package://staubli_description/meshes/visual/tete_extrusion.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 scale=0.001 0.001 0.001
Joints:
- added joint flange_to_tete: type fixed, parent flange, child tete_extrusion, origin xyz=0 0 -0.115 rpy=3.14159 3.14159 -2.0071
- added joint world_to_aeration: type fixed, parent world, child aeration, origin xyz=0.941 -0.725 0.0 rpy=0 0 0
- added joint world_to_controleur: type fixed, parent world, child controleur, origin xyz=0.470 4.040 0.0 rpy=0 0 0
- added joint world_to_silo: type fixed, parent world, child silo, origin xyz=0.700 1.000 0.0 rpy=0 0 0
- joint world_to_base: origin xyz=0 0 0 rpy=0 0 0 -> xyz=0 0 0 rpy=0 0 3.14159
